Commit message: fix(sim): V2.1 — unify spawn poses, optical frame_ids, isolated launch
Phase 0-1 (preflight + isolated launch):
- Add scene_v2_preflight.py: detect ROS/Gazebo conflicts
- Add run_scene_v2.sh: isolated ROS/Gazebo master, graceful cleanup

Phase 3 (unified geometry/spawn):
- gantry_v2.xacro: local coords only, spawn pose from launch (-x 0.78)
- object_v2.xacro: local coords only, spawn pose from launch (-x 0.72 -z 0.88)
- scene_v2.launch: actual spawn poses (not all zeros)

Phase 4 (dynamic object TF):
- Add object_pose_tf_v2.py: reads Gazebo pose, publishes world→object_frame
- Follows yaw rotation via set_model_state

Phase 6 (camera from YAML):
- spawn_cameras_v2.py: reads scene_v2.yaml for camera names/positions/target/profile
- No hardcoded CAMERAS/TARGET/PROFILE
- Camera body + lens + optical axis arrow visual

Phase 8 (optical frame_ids):
- Modify gazebo_ros_realsense plugin: custom colorFrameName/depthFrameName from SDF
- Verified: cam_front_left_color_optical_frame (not 'cam_front_leftcolor')
- Forward-compatible: ir1FrameName/ir2FrameName also supported

Verified:
- 0 errors (no joint1, no already exists, no exit 255)
- Controllers running
- frame_id matches optical TF convention

File: src/cr5_spray_sim/urdf/gantry_v2.xacro (robot description, xacro)
@@ -1,140 +1,123 @@
 <?xml version="1.0"?>
 <!--
-  Gantry V2: Four-post static frame, monolithic model
-  所有 visual/collision 在一个 link 中用 box 原语构建。
-  不加载 gazebo_ros_control。
+  Gantry V2: Monolithic static frame, local coords only.
+  World position applied by spawn_model pose.
+  Root link origin = bottom center of gantry frame.
+  Four pillars: ±Y = ±width/2, front/rear X = ±depth/2 from center.
 -->
 <robot name="gantry_v2" xmlns:xacro="http://ros.org/wiki/xacro">
-  <xacro:arg name="center_x" default="0.78"/>
   <xacro:arg name="width_y" default="1.45"/>
   <xacro:arg name="depth_x" default="0.75"/>
   <xacro:arg name="height" default="1.75"/>
   <xacro:arg name="beam" default="0.04"/>
-  <xacro:property name="cx" value="$(arg center_x)"/>
   <xacro:property name="wy" value="$(arg width_y)"/>
   <xacro:property name="dx" value="$(arg depth_x)"/>
   <xacro:property name="h" value="$(arg height)"/>
   <xacro:property name="b" value="$(arg beam)"/>
-  <xacro:property name="front_x" value="${cx - dx/2}"/>
-  <xacro:property name="rear_x" value="${cx + dx/2}"/>
-  <xacro:property name="left_y" value="${-wy/2}"/>
-  <xacro:property name="right_y" value="${wy/2}"/>
-  <material name="gantry_v2_gray">
+  <material name="gantry_gray">
     <color rgba="0.55 0.55 0.55 1"/>
   </material>
-  <!-- Single link containing all geometry -->
+  <!-- Root link: origin at bottom center of gantry frame -->
   <link name="gantry_v2_base">
     <inertial>
       <mass value="100.0"/>
       <inertia ixx="50.0" ixy="0" ixz="0" iyy="50.0" iyz="0" izz="50.0"/>
-      <origin xyz="${cx} 0 ${h/2}" rpy="0 0 0"/>
+      <origin xyz="0 0 ${h/2}" rpy="0 0 0"/>
     </inertial>
-    <!-- Four vertical pillars -->
     <!-- Front-left pillar -->
     <visual name="pillar_fl">
-      <origin xyz="${front_x} ${left_y} ${h/2}" rpy="0 0 0"/>
+      <origin xyz="${-dx/2} ${-wy/2} ${h/2}" rpy="0 0 0"/>
       <geometry><box size="${b} ${b} ${h}"/></geometry>
-      <material name="gantry_v2_gray"/>
+      <material name="gantry_gray"/>
     </visual>
     <collision name="pillar_fl_col">
-      <origin xyz="${front_x} ${left_y} ${h/2}" rpy="0 0 0"/>
+      <origin xyz="${-dx/2} ${-wy/2} ${h/2}" rpy="0 0 0"/>
       <geometry><box size="${b} ${b} ${h}"/></geometry>
     </collision>
     <!-- Front-right pillar -->
     <visual name="pillar_fr">
-      <origin xyz="${front_x} ${right_y} ${h/2}" rpy="0 0 0"/>
+      <origin xyz="${-dx/2} ${wy/2} ${h/2}" rpy="0 0 0"/>
       <geometry><box size="${b} ${b} ${h}"/></geometry>
-      <material name="gantry_v2_gray"/>
+      <material name="gantry_gray"/>
     </visual>
     <collision name="pillar_fr_col">
-      <origin xyz="${front_x} ${right_y} ${h/2}" rpy="0 0 0"/>
+      <origin xyz="${-dx/2} ${wy/2} ${h/2}" rpy="0 0 0"/>
       <geometry><box size="${b} ${b} ${h}"/></geometry>
     </collision>
     <!-- Rear-left pillar -->
     <visual name="pillar_rl">
-      <origin xyz="${rear_x} ${left_y} ${h/2}" rpy="0 0 0"/>
+      <origin xyz="${dx/2} ${-wy/2} ${h/2}" rpy="0 0 0"/>
       <geometry><box size="${b} ${b} ${h}"/></geometry>
-      <material name="gantry_v2_gray"/>
+      <material name="gantry_gray"/>
     </visual>
     <collision name="pillar_rl_col">
-      <origin xyz="${rear_x} ${left_y} ${h/2}" rpy="0 0 0"/>
+      <origin xyz="${dx/2} ${-wy/2} ${h/2}" rpy="0 0 0"/>
       <geometry><box size="${b} ${b} ${h}"/></geometry>
     </collision>
     <!-- Rear-right pillar -->
     <visual name="pillar_rr">
-      <origin xyz="${rear_x} ${right_y} ${h/2}" rpy="0 0 0"/>
+      <origin xyz="${dx/2} ${wy/2} ${h/2}" rpy="0 0 0"/>
       <geometry><box size="${b} ${b} ${h}"/></geometry>
-      <material name="gantry_v2_gray"/>
+      <material name="gantry_gray"/>
     </visual>
     <collision name="pillar_rr_col">
-      <origin xyz="${rear_x} ${right_y} ${h/2}" rpy="0 0 0"/>
+      <origin xyz="${dx/2} ${wy/2} ${h/2}" rpy="0 0 0"/>
       <geometry><box size="${b} ${b} ${h}"/></geometry>
     </collision>
-    <!-- Top beams: 4 sides forming closed rectangle -->
-    <!-- Front top beam (X direction, between front posts) -->
+    <!-- Top beams: 4 sides -->
     <visual name="beam_front">
-      <origin xyz="${cx} ${left_y} ${h - b/2}" rpy="0 0 0"/>
+      <origin xyz="${-dx/2} 0 ${h - b/2}" rpy="0 0 0"/>
       <geometry><box size="${dx} ${b} ${b}"/></geometry>
-      <material name="gantry_v2_gray"/>
+      <material name="gantry_gray"/>
     </visual>
     <collision name="beam_front_col">
-      <origin xyz="${cx} ${left_y} ${h - b/2}" rpy="0 0 0"/>
+      <origin xyz="${-dx/2} 0 ${h - b/2}" rpy="0 0 0"/>
       <geometry><box size="${dx} ${b} ${b}"/></geometry>
     </collision>
-    <!-- Rear top beam -->
     <visual name="beam_rear">
-      <origin xyz="${cx} ${right_y} ${h - b/2}" rpy="0 0 0"/>
+      <origin xyz="${dx/2} 0 ${h - b/2}" rpy="0 0 0"/>
       <geometry><box size="${dx} ${b} ${b}"/></geometry>
-      <material name="gantry_v2_gray"/>
+      <material name="gantry_gray"/>
     </visual>
     <collision name="beam_rear_col">
-      <origin xyz="${cx} ${right_y} ${h - b/2}" rpy="0 0 0"/>
+      <origin xyz="${dx/2} 0 ${h - b/2}" rpy="0 0 0"/>
       <geometry><box size="${dx} ${b} ${b}"/></geometry>
     </collision>
-    <!-- Left top beam (Y direction) -->
     <visual name="beam_left">
-      <origin xyz="${front_x} 0 ${h - b/2}" rpy="0 0 0"/>
+      <origin xyz="0 ${-wy/2} ${h - b/2}" rpy="0 0 0"/>
       <geometry><box size="${b} ${wy} ${b}"/></geometry>
-      <material name="gantry_v2_gray"/>
+      <material name="gantry_gray"/>
     </visual>
     <collision name="beam_left_col">
-      <origin xyz="${front_x} 0 ${h - b/2}" rpy="0 0 0"/>
+      <origin xyz="0 ${-wy/2} ${h - b/2}" rpy="0 0 0"/>
       <geometry><box size="${b} ${wy} ${b}"/></geometry>
     </collision>
-    <!-- Right top beam -->
     <visual name="beam_right">
-      <origin xyz="${rear_x} 0 ${h - b/2}" rpy="0 0 0"/>
+      <origin xyz="0 ${wy/2} ${h - b/2}" rpy="0 0 0"/>
       <geometry><box size="${b} ${wy} ${b}"/></geometry>
-      <material name="gantry_v2_gray"/>
+      <material name="gantry_gray"/>
     </visual>
     <collision name="beam_right_col">
-      <origin xyz="${rear_x} 0 ${h - b/2}" rpy="0 0 0"/>
+      <origin xyz="0 ${wy/2} ${h - b/2}" rpy="0 0 0"/>
       <geometry><box size="${b} ${wy} ${b}"/></geometry>
     </collision>
-    <!-- Base plates (feet) for each pillar -->
+    <!-- Base plates -->
     <visual name="foot_fl">
-      <origin xyz="${front_x} ${left_y} 0.01" rpy="0 0 0"/>
-      <geometry><box size="0.25 0.15 0.02"/></geometry>
-      <material name="gantry_v2_gray"/>
+      <origin xyz="${-dx/2} ${-wy/2} 0.01" rpy="0 0 0"/>
+      <geometry><box size="0.25 0.15 0.02"/></geometry><material name="gantry_gray"/>
     </visual>
     <visual name="foot_fr">
-      <origin xyz="${front_x} ${right_y} 0.01" rpy="0 0 0"/>
-      <geometry><box size="0.25 0.15 0.02"/></geometry>
-      <material name="gantry_v2_gray"/>
+      <origin xyz="${-dx/2} ${wy/2} 0.01" rpy="0 0 0"/>
+      <geometry><box size="0.25 0.15 0.02"/></geometry><material name="gantry_gray"/>
     </visual>
     <visual name="foot_rl">
-      <origin xyz="${rear_x} ${left_y} 0.01" rpy="0 0 0"/>
-      <geometry><box size="0.25 0.15 0.02"/></geometry>
-      <material name="gantry_v2_gray"/>
+      <origin xyz="${dx/2} ${-wy/2} 0.01" rpy="0 0 0"/>
+      <geometry><box size="0.25 0.15 0.02"/></geometry><material name="gantry_gray"/>
     </visual>
     <visual name="foot_rr">
-      <origin xyz="${rear_x} ${right_y} 0.01" rpy="0 0 0"/>
-      <geometry><box size="0.25 0.15 0.02"/></geometry>
-      <material name="gantry_v2_gray"/>
+      <origin xyz="${dx/2} ${wy/2} 0.01" rpy="0 0 0"/>
+      <geometry><box size="0.25 0.15 0.02"/></geometry><material name="gantry_gray"/>
     </visual>
   </link>
-  <!-- Static: not affected by gravity -->
-  <gazebo>
-    <static>true</static>
-  </gazebo>
+  <gazebo><static>true</static></gazebo>
 </robot>

File: src/cr5_spray_sim/urdf/object_v2.xacro (robot description, xacro)
@@ -1,118 +1,51 @@
 <?xml version="1.0"?>
 <!--
-  Object V2: Fixed workpiece, no ros_control, no rope simulation
-  Yaw rotation via set_model_state, not joint controller.
+  Object V2: Fixed workpiece, local coords only.
+  World position applied by spawn_model pose.
+  No ros_control. Yaw via set_model_state.
 -->
 <robot name="spray_object" xmlns:xacro="http://ros.org/wiki/xacro">
   <xacro:arg name="object_type" default="flat_panel"/>
-  <xacro:arg name="object_x" default="0.72"/>
-  <xacro:arg name="object_y" default="0.0"/>
-  <xacro:arg name="object_z" default="0.88"/>
   <xacro:property name="type" value="$(arg object_type)"/>
-  <xacro:property name="px" value="$(arg object_x)"/>
-  <xacro:property name="py" value="$(arg object_y)"/>
-  <xacro:property name="pz" value="$(arg object_z)"/>
-  <material name="object_v2_color">
-    <color rgba="0.6 0.6 0.7 1"/>
-  </material>
-  <!-- Object body in a single link with all geometry at origin -->
+  <material name="obj_v2_color"><color rgba="0.6 0.6 0.7 1"/></material>
+  <!-- Object frame at geometric center (local origin) -->
   <link name="object_frame"/>
   <xacro:if value="${type == 'flat_panel'}">
     <link name="object_body">
-      <inertial>
-        <mass value="0.5"/>
-        <inertia ixx="0.005" ixy="0" ixz="0" iyy="0.005" iyz="0" izz="0.005"/>
-      </inertial>
-      <visual>
-        <geometry><box size="0.30 0.02 0.30"/></geometry>
-        <material name="object_v2_color"/>
-      </visual>
-      <collision>
-        <geometry><box size="0.30 0.02 0.30"/></geometry>
-      </collision>
+      <inertial><mass value="0.5"/><inertia ixx="0.005" ixy="0" ixz="0" iyy="0.005" iyz="0" izz="0.005"/></inertial>
+      <visual><geometry><box size="0.30 0.02 0.30"/></geometry><material name="obj_v2_color"/></visual>
+      <collision><geometry><box size="0.30 0.02 0.30"/></geometry></collision>
     </link>
   </xacro:if>
   <xacro:if value="${type == 'cylinder_part'}">
     <link name="object_body">
-      <inertial>
-        <mass value="1.0"/>
-        <inertia ixx="0.01" ixy="0" ixz="0" iyy="0.01" iyz="0" izz="0.005"/>
-      </inertial>
-      <visual>
-        <origin xyz="0 0 0.175" rpy="0 0 0"/>
-        <geometry><cylinder radius="0.10" length="0.35"/></geometry>
-        <material name="object_v2_color"/>
-      </visual>
-      <collision>
-        <origin xyz="0 0 0.175" rpy="0 0 0"/>
-        <geometry><cylinder radius="0.10" length="0.35"/></geometry>
-      </collision>
+      <inertial><mass value="1.0"/><inertia ixx="0.01" ixy="0" ixz="0" iyy="0.01" iyz="0" izz="0.005"/></inertial>
+      <visual><origin xyz="0 0 0.175" rpy="0 0 0"/><geometry><cylinder radius="0.10" length="0.35"/></geometry><material name="obj_v2_color"/></visual>
+      <collision><origin xyz="0 0 0.175" rpy="0 0 0"/><geometry><cylinder radius="0.10" length="0.35"/></geometry></collision>
     </link>
   </xacro:if>
   <xacro:if value="${type == 'asymmetric_part_v2'}">
     <link name="object_body">
-      <inertial>
-        <mass value="0.8"/>
-        <inertia ixx="0.008" ixy="0" ixz="0" iyy="0.008" iyz="0" izz="0.005"/>
-        <origin xyz="0.03 0.01 0.08" rpy="0 0 0"/>
-      </inertial>
-      <!-- Programmatic asymmetric composite: L-shaped body + top block -->
-      <visual name="base_block">
-        <origin xyz="0 0 0.08" rpy="0 0 0"/>
-        <geometry><box size="0.20 0.15 0.16"/></geometry>
-        <material name="object_v2_color"/>
-      </visual>
-      <visual name="side_wing">
-        <origin xyz="0.12 0 0.06" rpy="0 0 0.3"/>
-        <geometry><box size="0.18 0.10 0.12"/></geometry>
-        <material name="object_v2_color"/>
-      </visual>
-      <visual name="top_nub">
-        <origin xyz="0.02 -0.04 0.17" rpy="0 0 0"/>
-        <geometry><cylinder radius="0.04" length="0.06"/></geometry>
-        <material name="object_v2_color"/>
-      </visual>
-      <visual name="front_notch">
-        <origin xyz="-0.08 0.05 0.04" rpy="0 0 0"/>
-        <geometry><box size="0.05 0.06 0.08"/></geometry>
-        <material name="object_v2_color"/>
-      </visual>
-      <!-- Collision approximates visual -->
-      <collision name="base_block_col">
-        <origin xyz="0 0 0.08" rpy="0 0 0"/>
-        <geometry><box size="0.20 0.15 0.16"/></geometry>
-      </collision>
-      <collision name="side_wing_col">
-        <origin xyz="0.12 0 0.06" rpy="0 0 0.3"/>
-        <geometry><box size="0.18 0.10 0.12"/></geometry>
-      </collision>
-      <!-- Ground-truth mesh = same geometry, can be exported to PLY -->
+      <inertial><mass value="0.8"/><inertia ixx="0.008" ixy="0" ixz="0" iyy="0.008" iyz="0" izz="0.005"/><origin xyz="0.03 0.01 0.08" rpy="0 0 0"/></inertial>
+      <visual name="base_block"><origin xyz="0 0 0.08" rpy="0 0 0"/><geometry><box size="0.20 0.15 0.16"/></geometry><material name="obj_v2_color"/></visual>
+      <visual name="side_wing"><origin xyz="0.12 0 0.06" rpy="0 0 0.3"/><geometry><box size="0.18 0.10 0.12"/></geometry><material name="obj_v2_color"/></visual>
+      <visual name="top_nub"><origin xyz="0.02 -0.04 0.17" rpy="0 0 0"/><geometry><cylinder radius="0.04" length="0.06"/></geometry><material name="obj_v2_color"/></visual>
+      <visual name="front_notch"><origin xyz="-0.08 0.05 0.04" rpy="0 0 0"/><geometry><box size="0.05 0.06 0.08"/></geometry><material name="obj_v2_color"/></visual>
+      <collision name="base_block_col"><origin xyz="0 0 0.08" rpy="0 0 0"/><geometry><box size="0.20 0.15 0.16"/></geometry></collision>
+      <collision name="side_wing_col"><origin xyz="0.12 0 0.06" rpy="0 0 0.3"/><geometry><box size="0.18 0.10 0.12"/></geometry></collision>
     </link>
   </xacro:if>
-  <!-- Fixed joint from frame to body -->
   <joint name="object_frame_to_body" type="fixed">
     <parent link="object_frame"/>
     <child link="object_body"/>
   </joint>
-  <!-- Suspension wire (visual only) -->
+  <!-- Visual wire -->
   <link name="object_wire">
-    <inertial>
-      <mass value="0.01"/>
-      <inertia ixx="0.00001" ixy="0" ixz="0" iyy="0.00001" iyz="0" izz="0.00001"/>
-    </inertial>
-    <visual>
-      <origin xyz="0 0 -0.10" rpy="0 0 0"/>
-      <geometry><cylinder radius="0.003" length="0.20"/></geometry>
-      <material name="object_v2_color"/>
-    </visual>
+    <inertial><mass value="0.01"/><inertia ixx="0.00001" ixy="0" ixz="0" iyy="0.00001" iyz="0" izz="0.00001"/></inertial>
+    <visual><origin xyz="0 0 -0.10" rpy="0 0 0"/><geometry><cylinder radius="0.003" length="0.20"/></geometry><material name="obj_v2_color"/></visual>
   </link>
   <joint name="object_frame_to_wire" type="fixed">
-    <parent link="object_frame"/>
-    <child link="object_wire"/>
-    <origin xyz="0 0 0" rpy="0 0 0"/>
+    <parent link="object_frame"/><child link="object_wire"/>
   </joint>
-  <!-- Static model - no ros_control! -->
-  <gazebo>
-    <static>true</static>
-  </gazebo>
+  <gazebo><static>true</static></gazebo>
 </robot>
