Commit message: fix(sim): rebuild top frame as closed rectangle, add block-combo target
- gantry_v2: fix top beam orientations — front/rear beams now run
  along Y (connecting left-right pillars), left/right beams run
  along X (connecting front-rear pillars). Add center cross-beam
  and suspension eyelet for clear hanging point.
- object_v2: add block_combo_part type — big block 0.28×0.18×0.30
  (blue) with small block 0.10×0.08×0.10 (orange) attached at
  top-right-front corner. Update flat_panel/cylinder colors.

File: src/cr5_spray_sim/urdf/gantry_v2.xacro (robot description, xacro)
@@ -1,8 +1,13 @@
 <?xml version="1.0"?>
 <!--
-  Gantry V2: Monolithic static frame, local coords only.
+  Gantry V2.2: Monolithic static frame with closed rectangular top.
   World position applied by spawn_model pose.
-  Root link origin = bottom center of gantry frame.
-  Four pillars: ±Y = ±width/2, front/rear X = ±depth/2 from center.
+  Root link origin = bottom center of gantry frame (ground level).
+  Structure:
+    4 pillars (square tubes) at corners
+    4 top beams forming a closed rectangle
+    1 center cross-beam for suspension point
+    4 base plates at pillar feet
+    1 hanging eyelet at center for wire attachment
 -->
 <robot name="gantry_v2" xmlns:xacro="http://ros.org/wiki/xacro">
@@ -15,107 +20,150 @@
   <xacro:property name="h" value="$(arg height)"/>
   <xacro:property name="b" value="$(arg beam)"/>
-  <material name="gantry_gray">
-    <color rgba="0.55 0.55 0.55 1"/>
+  <!-- Half-extents for placement -->
+  <xacro:property name="hx" value="${dx/2}"/>
+  <xacro:property name="hy" value="${wy/2}"/>
+  <!-- Materials: low-saturation demo palette -->
+  <material name="gantry_frame_gray">
+    <color rgba="0.52 0.52 0.52 1"/>
+  </material>
+  <material name="gantry_suspension_dark">
+    <color rgba="0.25 0.25 0.28 1"/>
   </material>
   <!-- Root link: origin at bottom center of gantry frame -->
   <link name="gantry_v2_base">
     <inertial>
-      <mass value="100.0"/>
-      <inertia ixx="50.0" ixy="0" ixz="0" iyy="50.0" iyz="0" izz="50.0"/>
+      <mass value="150.0"/>
+      <inertia ixx="80.0" ixy="0" ixz="0" iyy="80.0" iyz="0" izz="80.0"/>
       <origin xyz="0 0 ${h/2}" rpy="0 0 0"/>
     </inertial>
-    <!-- Front-left pillar -->
+    <!-- ===== Four Corner Pillars ===== -->
+    <!-- Front-Left -->
     <visual name="pillar_fl">
-      <origin xyz="${-dx/2} ${-wy/2} ${h/2}" rpy="0 0 0"/>
+      <origin xyz="${-hx} ${-hy} ${h/2}" rpy="0 0 0"/>
       <geometry><box size="${b} ${b} ${h}"/></geometry>
-      <material name="gantry_gray"/>
+      <material name="gantry_frame_gray"/>
     </visual>
     <collision name="pillar_fl_col">
-      <origin xyz="${-dx/2} ${-wy/2} ${h/2}" rpy="0 0 0"/>
+      <origin xyz="${-hx} ${-hy} ${h/2}" rpy="0 0 0"/>
       <geometry><box size="${b} ${b} ${h}"/></geometry>
     </collision>
-    <!-- Front-right pillar -->
+    <!-- Front-Right -->
     <visual name="pillar_fr">
-      <origin xyz="${-dx/2} ${wy/2} ${h/2}" rpy="0 0 0"/>
+      <origin xyz="${-hx} ${hy} ${h/2}" rpy="0 0 0"/>
       <geometry><box size="${b} ${b} ${h}"/></geometry>
-      <material name="gantry_gray"/>
+      <material name="gantry_frame_gray"/>
     </visual>
     <collision name="pillar_fr_col">
-      <origin xyz="${-dx/2} ${wy/2} ${h/2}" rpy="0 0 0"/>
+      <origin xyz="${-hx} ${hy} ${h/2}" rpy="0 0 0"/>
       <geometry><box size="${b} ${b} ${h}"/></geometry>
     </collision>
-    <!-- Rear-left pillar -->
+    <!-- Rear-Left -->
     <visual name="pillar_rl">
-      <origin xyz="${dx/2} ${-wy/2} ${h/2}" rpy="0 0 0"/>
+      <origin xyz="${hx} ${-hy} ${h/2}" rpy="0 0 0"/>
       <geometry><box size="${b} ${b} ${h}"/></geometry>
-      <material name="gantry_gray"/>
+      <material name="gantry_frame_gray"/>
     </visual>
     <collision name="pillar_rl_col">
-      <origin xyz="${dx/2} ${-wy/2} ${h/2}" rpy="0 0 0"/>
+      <origin xyz="${hx} ${-hy} ${h/2}" rpy="0 0 0"/>
       <geometry><box size="${b} ${b} ${h}"/></geometry>
     </collision>
-    <!-- Rear-right pillar -->
+    <!-- Rear-Right -->
     <visual name="pillar_rr">
-      <origin xyz="${dx/2} ${wy/2} ${h/2}" rpy="0 0 0"/>
+      <origin xyz="${hx} ${hy} ${h/2}" rpy="0 0 0"/>
       <geometry><box size="${b} ${b} ${h}"/></geometry>
-      <material name="gantry_gray"/>
+      <material name="gantry_frame_gray"/>
     </visual>
     <collision name="pillar_rr_col">
-      <origin xyz="${dx/2} ${wy/2} ${h/2}" rpy="0 0 0"/>
+      <origin xyz="${hx} ${hy} ${h/2}" rpy="0 0 0"/>
       <geometry><box size="${b} ${b} ${h}"/></geometry>
     </collision>
-    <!-- Top beams: 4 sides -->
+    <!-- ===== Top Beams: Closed Rectangle ===== -->
+    <!--
+      Beam naming: connects FL↔FR (front), FL↔RL (left), FR↔RR (right), RL↔RR (rear).
+      Front/Rear beams run along Y; Left/Right beams run along X.
+    -->
+    <!-- Front beam: FL ↔ FR  (along Y at X=-hx) -->
     <visual name="beam_front">
-      <origin xyz="${-dx/2} 0 ${h - b/2}" rpy="0 0 0"/>
-      <geometry><box size="${dx} ${b} ${b}"/></geometry>
-      <material name="gantry_gray"/>
+      <origin xyz="${-hx} 0 ${h - b/2}" rpy="0 0 0"/>
+      <geometry><box size="${b} ${wy} ${b}"/></geometry>
+      <material name="gantry_frame_gray"/>
     </visual>
     <collision name="beam_front_col">
-      <origin xyz="${-dx/2} 0 ${h - b/2}" rpy="0 0 0"/>
+      <origin xyz="${-hx} 0 ${h - b/2}" rpy="0 0 0"/>
+      <geometry><box size="${b} ${wy} ${b}"/></geometry>
+    </collision>
+    <!-- Rear beam: RL ↔ RR  (along Y at X=+hx) -->
+    <visual name="beam_rear">
+      <origin xyz="${hx} 0 ${h - b/2}" rpy="0 0 0"/>
+      <geometry><box size="${b} ${wy} ${b}"/></geometry>
+      <material name="gantry_frame_gray"/>
+    </visual>
+    <collision name="beam_rear_col">
+      <origin xyz="${hx} 0 ${h - b/2}" rpy="0 0 0"/>
+      <geometry><box size="${b} ${wy} ${b}"/></geometry>
+    </collision>
+    <!-- Left beam: FL ↔ RL  (along X at Y=-hy) -->
+    <visual name="beam_left">
+      <origin xyz="0 ${-hy} ${h - b/2}" rpy="0 0 0"/>
+      <geometry><box size="${dx} ${b} ${b}"/></geometry>
+      <material name="gantry_frame_gray"/>
+    </visual>
+    <collision name="beam_left_col">
+      <origin xyz="0 ${-hy} ${h - b/2}" rpy="0 0 0"/>
       <geometry><box size="${dx} ${b} ${b}"/></geometry>
     </collision>
-    <visual name="beam_rear">
-      <origin xyz="${dx/2} 0 ${h - b/2}" rpy="0 0 0"/>
+    <!-- Right beam: FR ↔ RR  (along X at Y=+hy) -->
+    <visual name="beam_right">
+      <origin xyz="0 ${hy} ${h - b/2}" rpy="0 0 0"/>
       <geometry><box size="${dx} ${b} ${b}"/></geometry>
-      <material name="gantry_gray"/>
+      <material name="gantry_frame_gray"/>
     </visual>
-    <collision name="beam_rear_col">
-      <origin xyz="${dx/2} 0 ${h - b/2}" rpy="0 0 0"/>
+    <collision name="beam_right_col">
+      <origin xyz="0 ${hy} ${h - b/2}" rpy="0 0 0"/>
       <geometry><box size="${dx} ${b} ${b}"/></geometry>
     </collision>
-    <visual name="beam_left">
-      <origin xyz="0 ${-wy/2} ${h - b/2}" rpy="0 0 0"/>
-      <geometry><box size="${b} ${wy} ${b}"/></geometry>
-      <material name="gantry_gray"/>
+    <!-- ===== Center Cross-Beam (X-direction, at Y=0) ===== -->
+    <visual name="beam_center">
+      <origin xyz="0 0 ${h - b/2}" rpy="0 0 0"/>
+      <geometry><box size="${dx} ${b*0.6} ${b}"/></geometry>
+      <material name="gantry_frame_gray"/>
     </visual>
-    <collision name="beam_left_col">
-      <origin xyz="0 ${-wy/2} ${h - b/2}" rpy="0 0 0"/>
-      <geometry><box size="${b} ${wy} ${b}"/></geometry>
+    <collision name="beam_center_col">
+      <origin xyz="0 0 ${h - b/2}" rpy="0 0 0"/>
+      <geometry><box size="${dx} ${b*0.6} ${b}"/></geometry>
     </collision>
-    <visual name="beam_right">
-      <origin xyz="0 ${wy/2} ${h - b/2}" rpy="0 0 0"/>
-      <geometry><box size="${b} ${wy} ${b}"/></geometry>
-      <material name="gantry_gray"/>
+    <!-- ===== Center Suspension Eyelet (hanging point) ===== -->
+    <!-- Small bracket hanging below center cross-beam -->
+    <visual name="eyelet_bracket">
+      <origin xyz="0 0 ${h - b*1.8}" rpy="0 0 0"/>
+      <geometry><box size="${b*1.2} ${b*1.2} ${b*0.8}"/></geometry>
+      <material name="gantry_suspension_dark"/>
     </visual>
-    <collision name="beam_right_col">
-      <origin xyz="0 ${wy/2} ${h - b/2}" rpy="0 0 0"/>
-      <geometry><box size="${b} ${wy} ${b}"/></geometry>
-    </collision>
-    <!-- Base plates -->
+    <!-- Ring/eyelet for wire attachment -->
+    <visual name="eyelet_ring">
+      <origin xyz="0 0 ${h - b*2.6}" rpy="0 0 0"/>
+      <geometry><cylinder radius="${b*0.9}" length="${b*0.3}"/></geometry>
+      <material name="gantry_suspension_dark"/>
+    </visual>
+    <!-- ===== Base Plates (feet) ===== -->
     <visual name="foot_fl">
-      <origin xyz="${-dx/2} ${-wy/2} 0.01" rpy="0 0 0"/>
-      <geometry><box size="0.25 0.15 0.02"/></geometry><material name="gantry_gray"/>
+      <origin xyz="${-hx} ${-hy} 0.01" rpy="0 0 0"/>
+      <geometry><box size="0.25 0.15 0.02"/></geometry>
+      <material name="gantry_frame_gray"/>
     </visual>
     <visual name="foot_fr">
-      <origin xyz="${-dx/2} ${wy/2} 0.01" rpy="0 0 0"/>
-      <geometry><box size="0.25 0.15 0.02"/></geometry><material name="gantry_gray"/>
+      <origin xyz="${-hx} ${hy} 0.01" rpy="0 0 0"/>
+      <geometry><box size="0.25 0.15 0.02"/></geometry>
+      <material name="gantry_frame_gray"/>
     </visual>
     <visual name="foot_rl">
-      <origin xyz="${dx/2} ${-wy/2} 0.01" rpy="0 0 0"/>
-      <geometry><box size="0.25 0.15 0.02"/></geometry><material name="gantry_gray"/>
+      <origin xyz="${hx} ${-hy} 0.01" rpy="0 0 0"/>
+      <geometry><box size="0.25 0.15 0.02"/></geometry>
+      <material name="gantry_frame_gray"/>
     </visual>
     <visual name="foot_rr">
-      <origin xyz="${dx/2} ${wy/2} 0.01" rpy="0 0 0"/>
-      <geometry><box size="0.25 0.15 0.02"/></geometry><material name="gantry_gray"/>
+      <origin xyz="${hx} ${hy} 0.01" rpy="0 0 0"/>
+      <geometry><box size="0.25 0.15 0.02"/></geometry>
+      <material name="gantry_frame_gray"/>
     </visual>
   </link>

File: src/cr5_spray_sim/urdf/object_v2.xacro (robot description, xacro)
@@ -1,35 +1,91 @@
 <?xml version="1.0"?>
 <!--
-  Object V2: Fixed workpiece, local coords only.
+  Object V2.2: Fixed workpiece with demo colors.
   World position applied by spawn_model pose.
   No ros_control. Yaw via set_model_state.
+  Types:
+    flat_panel         — thin plate 0.30×0.02×0.30
+    cylinder_part      — cylinder r=0.10 h=0.35
+    block_combo_part   — big block 0.28×0.18×0.30 + small block 0.10×0.08×0.10
 -->
 <robot name="spray_object" xmlns:xacro="http://ros.org/wiki/xacro">
-  <xacro:arg name="object_type" default="flat_panel"/>
+  <xacro:arg name="object_type" default="block_combo_part"/>
   <xacro:property name="type" value="$(arg object_type)"/>
-  <material name="obj_v2_color"><color rgba="0.6 0.6 0.7 1"/></material>
+  <!-- Demo color palette -->
+  <material name="obj_main_blue">   <!-- big block / main body -->
+    <color rgba="0.10 0.35 0.75 1"/>
+  </material>
+  <material name="obj_accent_orange"><!-- small block / direction feature -->
+    <color rgba="0.92 0.45 0.08 1"/>
+  </material>
+  <material name="obj_wire_dark">   <!-- suspension wire -->
+    <color rgba="0.18 0.18 0.20 1"/>
+  </material>
+  <material name="obj_flat_gray">   <!-- flat_panel fallback -->
+    <color rgba="0.55 0.55 0.60 1"/>
+  </material>
+  <material name="obj_cylinder_teal"><!-- cylinder fallback -->
+    <color rgba="0.15 0.55 0.55 1"/>
+  </material>
   <!-- Object frame at geometric center (local origin) -->
   <link name="object_frame"/>
+  <!-- ===== flat_panel ===== -->
   <xacro:if value="${type == 'flat_panel'}">
     <link name="object_body">
       <inertial><mass value="0.5"/><inertia ixx="0.005" ixy="0" ixz="0" iyy="0.005" iyz="0" izz="0.005"/></inertial>
-      <visual><geometry><box size="0.30 0.02 0.30"/></geometry><material name="obj_v2_color"/></visual>
+      <visual><geometry><box size="0.30 0.02 0.30"/></geometry><material name="obj_flat_gray"/></visual>
       <collision><geometry><box size="0.30 0.02 0.30"/></geometry></collision>
     </link>
   </xacro:if>
+  <!-- ===== cylinder_part ===== -->
   <xacro:if value="${type == 'cylinder_part'}">
     <link name="object_body">
       <inertial><mass value="1.0"/><inertia ixx="0.01" ixy="0" ixz="0" iyy="0.01" iyz="0" izz="0.005"/></inertial>
-      <visual><origin xyz="0 0 0.175" rpy="0 0 0"/><geometry><cylinder radius="0.10" length="0.35"/></geometry><material name="obj_v2_color"/></visual>
+      <visual><origin xyz="0 0 0.175" rpy="0 0 0"/><geometry><cylinder radius="0.10" length="0.35"/></geometry><material name="obj_cylinder_teal"/></visual>
       <collision><origin xyz="0 0 0.175" rpy="0 0 0"/><geometry><cylinder radius="0.10" length="0.35"/></geometry></collision>
     </link>
   </xacro:if>
+  <!-- ===== block_combo_part: big block + small block ===== -->
+  <xacro:if value="${type == 'block_combo_part'}">
+    <link name="object_body">
+      <inertial>
+        <mass value="1.2"/>
+        <!-- Combined inertia estimated for two blocks -->
+        <inertia ixx="0.015" ixy="0" ixz="0" iyy="0.012" iyz="0" izz="0.010"/>
+        <origin xyz="0.02 0.0 0.14" rpy="0 0 0"/>
+      </inertial>
+      <!-- Big block: main body (blue) -->
+      <!-- size: 0.28(X) × 0.18(Y) × 0.30(Z), center at z=0.15 -->
+      <visual name="big_block">
+        <origin xyz="0 0 0.15" rpy="0 0 0"/>
+        <geometry><box size="0.28 0.18 0.30"/></geometry>
+        <material name="obj_main_blue"/>
+      </visual>
+      <collision name="big_block_col">
+        <origin xyz="0 0 0.15" rpy="0 0 0"/>
+        <geometry><box size="0.28 0.18 0.30"/></geometry>
+      </collision>
+      <!-- Small block: direction feature (orange), attached to top-right-front -->
+      <!-- size: 0.10(X) × 0.08(Y) × 0.10(Z) -->
+      <!-- Position: front-right top corner of big block -->
+      <visual name="small_block">
+        <origin xyz="0.09 0.07 0.32" rpy="0 0 0"/>
+        <geometry><box size="0.10 0.08 0.10"/></geometry>
+        <material name="obj_accent_orange"/>
+      </visual>
+      <collision name="small_block_col">
+        <origin xyz="0.09 0.07 0.32" rpy="0 0 0"/>
+        <geometry><box size="0.10 0.08 0.10"/></geometry>
+      </collision>
+    </link>
+  </xacro:if>
+  <!-- ===== asymmetric_part_v2 (legacy) ===== -->
   <xacro:if value="${type == 'asymmetric_part_v2'}">
     <link name="object_body">
       <inertial><mass value="0.8"/><inertia ixx="0.008" ixy="0" ixz="0" iyy="0.008" iyz="0" izz="0.005"/><origin xyz="0.03 0.01 0.08" rpy="0 0 0"/></inertial>
-      <visual name="base_block"><origin xyz="0 0 0.08" rpy="0 0 0"/><geometry><box size="0.20 0.15 0.16"/></geometry><material name="obj_v2_color"/></visual>
-      <visual name="side_wing"><origin xyz="0.12 0 0.06" rpy="0 0 0.3"/><geometry><box size="0.18 0.10 0.12"/></geometry><material name="obj_v2_color"/></visual>
-      <visual name="top_nub"><origin xyz="0.02 -0.04 0.17" rpy="0 0 0"/><geometry><cylinder radius="0.04" length="0.06"/></geometry><material name="obj_v2_color"/></visual>
-      <visual name="front_notch"><origin xyz="-0.08 0.05 0.04" rpy="0 0 0"/><geometry><box size="0.05 0.06 0.08"/></geometry><material name="obj_v2_color"/></visual>
+      <visual name="base_block"><origin xyz="0 0 0.08" rpy="0 0 0"/><geometry><box size="0.20 0.15 0.16"/></geometry><material name="obj_main_blue"/></visual>
+      <visual name="side_wing"><origin xyz="0.12 0 0.06" rpy="0 0 0.3"/><geometry><box size="0.18 0.10 0.12"/></geometry><material name="obj_accent_orange"/></visual>
+      <visual name="top_nub"><origin xyz="0.02 -0.04 0.17" rpy="0 0 0"/><geometry><cylinder radius="0.04" length="0.06"/></geometry><material name="obj_accent_orange"/></visual>
+      <visual name="front_notch"><origin xyz="-0.08 0.05 0.04" rpy="0 0 0"/><geometry><box size="0.05 0.06 0.08"/></geometry><material name="obj_main_blue"/></visual>
       <collision name="base_block_col"><origin xyz="0 0 0.08" rpy="0 0 0"/><geometry><box size="0.20 0.15 0.16"/></geometry></collision>
       <collision name="side_wing_col"><origin xyz="0.12 0 0.06" rpy="0 0 0.3"/><geometry><box size="0.18 0.10 0.12"/></geometry></collision>
@@ -40,8 +96,12 @@
     <child link="object_body"/>
   </joint>
-  <!-- Visual wire -->
+  <!-- Visual suspension wire (dark, from object_frame up to gantry eyelet) -->
   <link name="object_wire">
     <inertial><mass value="0.01"/><inertia ixx="0.00001" ixy="0" ixz="0" iyy="0.00001" iyz="0" izz="0.00001"/></inertial>
-    <visual><origin xyz="0 0 -0.10" rpy="0 0 0"/><geometry><cylinder radius="0.003" length="0.20"/></geometry><material name="obj_v2_color"/></visual>
+    <visual>
+      <origin xyz="0 0 -0.10" rpy="0 0 0"/>
+      <geometry><cylinder radius="0.003" length="0.20"/></geometry>
+      <material name="obj_wire_dark"/>
+    </visual>
   </link>
   <joint name="object_frame_to_wire" type="fixed">
