Commit message: fix(sim): mount spray gun on actual Link6 flange interface
V3.2.1 使用旧 Tool_end 坐标 (-0.00683, 0.150178, 0.22462) 安装喷枪，
导致喷枪悬离法兰 ~22cm。V3.3 修正为从 Link6 原点安装：

- mount_xyz: (0, 0, 0.010) — 适配板背面贴合法兰面
- Visual-only 第一阶段: 零附加质量，无 collision
- 所有 visual 合并到单个 spray_gun_assembly link
- 仅 spray_nozzle_frame 作为 TF 参考系
- 备选: enable_spray_tool=false 时保留空 nozzle_frame fallback

File: src/cr5_spray_sim/urdf/cr5_sim.urdf.xacro (robot description, xacro)
@@ -13,4 +13,5 @@
   <xacro:arg name="sim_damping" default="0.5"/>
   <xacro:arg name="sim_friction" default="0.1"/>
+  <xacro:arg name="enable_spray_tool" default="true"/>
   <xacro:property name="effort_val" value="$(arg sim_effort)"/>
   <xacro:property name="velocity_val" value="$(arg sim_velocity)"/>
@@ -191,25 +192,28 @@
     <dynamics damping="${damping_val}" friction="${friction_val}"/>
   </joint>
-  <!-- ===== Spray Tool Frames (sim overlay) ===== -->
-  <!-- spray_tool_mount: attaches to Link6 flange -->
-  <link name="spray_tool_mount">
-    <inertial>
-      <mass value="0.05"/>
-      <inertia ixx="0.0001" ixy="0" ixz="0" iyy="0.0001" iyz="0" izz="0.0001"/>
-      <origin xyz="0 0 0" rpy="0 0 0"/>
-    </inertial>
-  </link>
-  <joint name="spray_tool_mount_joint" type="fixed">
-    <parent link="Link6"/>
-    <child link="spray_tool_mount"/>
-    <origin xyz="-0.00683 0.150178 0.22462" rpy="-0.0044 0.04684 -1.631"/>
-  </joint>
-  <!-- spray_nozzle_frame: +Z points from nozzle toward surface -->
-  <link name="spray_nozzle_frame"/>
-  <joint name="spray_nozzle_joint" type="fixed">
-    <parent link="spray_tool_mount"/>
-    <child link="spray_nozzle_frame"/>
-    <origin xyz="0 0 0.05" rpy="0 0 0"/>
-  </joint>
+  <!-- ===== Spray Tool V3.3 (visual-only, controlled by enable_spray_tool) ===== -->
+  <!--
+    安装位置: Link6 法兰面 (Link6 原点)，非旧 Tool_end。
+    适配板厚 0.020m，背面贴合法兰面 → mount_xyz.z = 0.010。
+    详见 config/spray_tool_mount_v33.yaml。
+    第一阶段: visual-only (零附加质量，无 collision)。
+    后续阶段可逐步加入 collision 和 payload mass。
+  -->
+  <xacro:if value="$(arg enable_spray_tool)">
+    <xacro:include filename="$(find cr5_spray_sim)/urdf/spray_gun_v33.xacro"/>
+    <xacro:spray_gun_v33 parent="Link6"
+        mount_xyz="0 0 0.010"
+        mount_rpy="0 0 0"
+        prefix="spray"/>
+  </xacro:if>
+  <!-- 无喷枪时的 fallback: 保留空 nozzle_frame 供 TF 查询 -->
+  <xacro:unless value="$(arg enable_spray_tool)">
+    <link name="spray_nozzle_frame"/>
+    <joint name="spray_nozzle_frame_fallback" type="fixed">
+      <parent link="Link6"/>
+      <child link="spray_nozzle_frame"/>
+      <origin xyz="0 0 0.125" rpy="0 0 0"/>
+    </joint>
+  </xacro:unless>
   <!-- wrist_d455_mount: wrist camera mount on Link6 -->
   <link name="wrist_d455_mount"/>

Commit message: fix(sim): embed spray gun visuals directly in Link6
V3.3.1 喷枪可见性修复:

- 删除 V3.3 的 spray_gun_assembly 独立 link (零质量/零惯量不可靠)
- 所有喷枪 visual 直接放入 Link6，属于同一 Gazebo 刚体
- 仅保留 spray_nozzle_frame 空 link 作为 TF 参考
- 新增绿色喷嘴轴指示器 (debug visual)
- Visuals-only xacro macro (spray_gun_v331_visuals.xacro)
- enable_spray_tool=true: 7 visual 并入 Link6, nozzle_frame 在 z=0.125
- enable_spray_tool=false: 仅 nozzle_frame fallback

File: src/cr5_spray_sim/urdf/cr5_sim.urdf.xacro (robot description, xacro)
@@ -14,4 +14,8 @@
   <xacro:arg name="sim_friction" default="0.1"/>
   <xacro:arg name="enable_spray_tool" default="true"/>
+  <!-- V3.3.1: 喷枪 visual macro (需在 Link6 之前 include) -->
+  <xacro:if value="$(arg enable_spray_tool)">
+    <xacro:include filename="$(find cr5_spray_sim)/urdf/spray_gun_v331_visuals.xacro"/>
+  </xacro:if>
   <xacro:property name="effort_val" value="$(arg sim_effort)"/>
   <xacro:property name="velocity_val" value="$(arg sim_velocity)"/>
@@ -183,4 +187,8 @@
       <geometry><mesh filename="package://dobot_description/meshes/cr5/Link6.dae"/></geometry>
     </collision>
+    <!-- V3.3.1: 喷枪 visual 直接并入 Link6 (同一 Gazebo 刚体, 不会漂移或消失) -->
+    <xacro:if value="$(arg enable_spray_tool)">
+      <xacro:spray_gun_v331_visuals prefix="spray"/>
+    </xacro:if>
   </link>
   <joint name="joint6" type="revolute">
@@ -192,28 +200,18 @@
     <dynamics damping="${damping_val}" friction="${friction_val}"/>
   </joint>
-  <!-- ===== Spray Tool V3.3 (visual-only, controlled by enable_spray_tool) ===== -->
+  <!-- ===== Spray Tool V3.3.1 ===== -->
   <!--
-    安装位置: Link6 法兰面 (Link6 原点)，非旧 Tool_end。
-    适配板厚 0.020m，背面贴合法兰面 → mount_xyz.z = 0.010。
-    详见 config/spray_tool_mount_v33.yaml。
-    第一阶段: visual-only (零附加质量，无 collision)。
-    后续阶段可逐步加入 collision 和 payload mass。
+    喷枪 visual 已直接并入 Link6 (同 Gazebo 刚体)。
+    此处只保留 spray_nozzle_frame 作为 TF 参考系。
+    安装位置: Link6 法兰原点。nozzle_frame 在喷嘴出口 z=0.125m。
   -->
-  <xacro:if value="$(arg enable_spray_tool)">
-    <xacro:include filename="$(find cr5_spray_sim)/urdf/spray_gun_v33.xacro"/>
-    <xacro:spray_gun_v33 parent="Link6"
-        mount_xyz="0 0 0.010"
-        mount_rpy="0 0 0"
-        prefix="spray"/>
-  </xacro:if>
-  <!-- 无喷枪时的 fallback: 保留空 nozzle_frame 供 TF 查询 -->
-  <xacro:unless value="$(arg enable_spray_tool)">
-    <link name="spray_nozzle_frame"/>
-    <joint name="spray_nozzle_frame_fallback" type="fixed">
-      <parent link="Link6"/>
-      <child link="spray_nozzle_frame"/>
-      <origin xyz="0 0 0.125" rpy="0 0 0"/>
-    </joint>
-  </xacro:unless>
+  <!-- spray_nozzle_frame: +Z = 喷射方向 (TF 查询用) -->
+  <link name="spray_nozzle_frame"/>
+  <joint name="spray_nozzle_frame_joint" type="fixed">
+    <parent link="Link6"/>
+    <child link="spray_nozzle_frame"/>
+    <!-- 喷嘴总长: 适配板半厚(0.010) + 枪体(0.075) + 喷嘴(0.040) = 0.125 -->
+    <origin xyz="0 0 0.125" rpy="0 0 0"/>
+  </joint>
   <!-- wrist_d455_mount: wrist camera mount on Link6 -->
   <link name="wrist_d455_mount"/>
