Commit message: fix(xacro): correct arg syntax in fixed_rgbd_camera.urdf.xacro
- Changed ${arg_name} → $(arg name) (xacro arg reference syntax)
- Verified: xacro command generates valid URDF with 19 link/sensor/plugin elements
- Headless simulation: CAMERA_COLOR_3_OF_3_PASS, CAMERA_DEPTH_3_OF_3_PASS

File: src/cr5_spray_sim/urdf/fixed_rgbd_camera.urdf.xacro (robot description, xacro)
@@ -14,9 +14,9 @@
   <xacro:arg name="color_hfov" default="1.2112585"/>
   <xacro:arg name="depth_hfov" default="1.2112585"/>
-  <material name="${arg_name}_body"><color rgba="0.25 0.25 0.25 1"/></material>
-  <material name="${arg_name}_lens"><color rgba="0.05 0.05 0.05 1"/></material>
-  <material name="${arg_name}_axis"><color rgba="1 0.15 0.15 1"/></material>
-  <material name="${arg_name}_up_mark"><color rgba="0.15 0.7 0.15 1"/></material>
-  <link name="${arg_name}_link">
+  <material name="$(arg name)_body"><color rgba="0.25 0.25 0.25 1"/></material>
+  <material name="$(arg name)_lens"><color rgba="0.05 0.05 0.05 1"/></material>
+  <material name="$(arg name)_axis"><color rgba="1 0.15 0.15 1"/></material>
+  <material name="$(arg name)_up_mark"><color rgba="0.15 0.7 0.15 1"/></material>
+  <link name="$(arg name)_link">
     <inertial>
       <mass value="0.05"/>
@@ -26,38 +26,38 @@
       <origin xyz="0 0 0" rpy="0 0 0"/>
       <geometry><box size="0.03 0.09 0.025"/></geometry>
-      <material name="${arg_name}_body"/>
+      <material name="$(arg name)_body"/>
     </visual>
     <visual name="lens">
       <origin xyz="0.015 0 0" rpy="0 1.5708 0"/>
       <geometry><cylinder radius="0.010" length="0.004"/></geometry>
-      <material name="${arg_name}_lens"/>
+      <material name="$(arg name)_lens"/>
     </visual>
     <visual name="axis">
       <origin xyz="0.025 0 0" rpy="0 1.5708 0"/>
       <geometry><cylinder radius="0.002" length="0.05"/></geometry>
-      <material name="${arg_name}_axis"/>
+      <material name="$(arg name)_axis"/>
     </visual>
     <visual name="up_dot">
       <origin xyz="0 0 0.013" rpy="0 0 0"/>
       <geometry><cylinder radius="0.004" length="0.003"/></geometry>
-      <material name="${arg_name}_up_mark"/>
+      <material name="$(arg name)_up_mark"/>
     </visual>
   </link>
-  <link name="${arg_name}_color_optical_frame"/>
-  <joint name="${arg_name}_color_optical_joint" type="fixed">
-    <parent link="${arg_name}_link"/>
-    <child link="${arg_name}_color_optical_frame"/>
+  <link name="$(arg name)_color_optical_frame"/>
+  <joint name="$(arg name)_color_optical_joint" type="fixed">
+    <parent link="$(arg name)_link"/>
+    <child link="$(arg name)_color_optical_frame"/>
     <origin xyz="0 0 0" rpy="-1.5708 0 -1.5708"/>
   </joint>
-  <link name="${arg_name}_depth_optical_frame"/>
-  <joint name="${arg_name}_depth_optical_joint" type="fixed">
-    <parent link="${arg_name}_link"/>
-    <child link="${arg_name}_depth_optical_frame"/>
+  <link name="$(arg name)_depth_optical_frame"/>
+  <joint name="$(arg name)_depth_optical_joint" type="fixed">
+    <parent link="$(arg name)_link"/>
+    <child link="$(arg name)_depth_optical_frame"/>
     <origin xyz="0 0 0" rpy="-1.5708 0 -1.5708"/>
   </joint>
-  <gazebo reference="${arg_name}_link">
+  <gazebo reference="$(arg name)_link">
     <self_collide>0</self_collide>
-    <sensor name="${arg_name}color" type="camera">
-      <camera name="${arg_name}">
+    <sensor name="$(arg name)color" type="camera">
+      <camera name="$(arg name)">
         <horizontal_fov>$(arg color_hfov)</horizontal_fov>
         <image>
@@ -73,6 +73,6 @@
       <visualize>false</visualize>
     </sensor>
-    <sensor name="${arg_name}depth" type="depth">
-      <camera name="${arg_name}">
+    <sensor name="$(arg name)depth" type="depth">
+      <camera name="$(arg name)">
         <horizontal_fov>$(arg depth_hfov)</horizontal_fov>
         <image>
@@ -88,6 +88,6 @@
       <visualize>false</visualize>
     </sensor>
-    <sensor name="${arg_name}ired1" type="camera">
-      <camera name="${arg_name}">
+    <sensor name="$(arg name)ired1" type="camera">
+      <camera name="$(arg name)">
         <horizontal_fov>1.48702</horizontal_fov>
         <image><width>160</width><height>120</height><format>L_INT8</format></image>
@@ -96,6 +96,6 @@
       <always_on>1</always_on><update_rate>2</update_rate><visualize>false</visualize>
     </sensor>
-    <sensor name="${arg_name}ired2" type="camera">
-      <camera name="${arg_name}">
+    <sensor name="$(arg name)ired2" type="camera">
+      <camera name="$(arg name)">
         <horizontal_fov>1.48702</horizontal_fov>
         <image><width>160</width><height>120</height><format>L_INT8</format></image>
@@ -106,8 +106,8 @@
   </gazebo>
   <gazebo>
-    <plugin name="${arg_name}" filename="librealsense_gazebo_plugin.so">
-      <prefix>${arg_name}</prefix>
-      <colorFrameName>${arg_name}_color_optical_frame</colorFrameName>
-      <depthFrameName>${arg_name}_depth_optical_frame</depthFrameName>
+    <plugin name="$(arg name)" filename="librealsense_gazebo_plugin.so">
+      <prefix>$(arg name)</prefix>
+      <colorFrameName>$(arg name)_color_optical_frame</colorFrameName>
+      <depthFrameName>$(arg name)_depth_optical_frame</depthFrameName>
     </plugin>
   </gazebo>
